File: fab/kicad/controller_pcb/controller_pcb.kicad_pcb (KiCad board)
At the start: 4 copper layers, 102.2 x 74.4 mm, 54 parts, among them J1 Screw_Terminal_01x04, J10 1935161, J11 Screw_Terminal_01x06, J2 Screw_Terminal_01x03, J3 Screw_Terminal_01x03, J4 Screw_Terminal_01x03, J5 Screw_Terminal_01x06, J6 Screw_Terminal_01x06, J7 Screw_Terminal_01x02, J8 1935161, J9 Screw_Terminal_01x02, Q1 IRLZ44N, U1 TPS55289RYQR, U2 TPS55289RYQR, U3 DS3231SN, U4 BK-912-TR

Commit message: v2 of PCB
Parts:
- added R10: CRCW0402100KFKED, extracted:RESC1005X40N, F.Cu at (129.2, 100.5)
- added R11: CFM14JT8K20, Resistor_THT:R_Axial_DIN0204_L3.6mm_D1.6mm_P5.08mm_Horizontal, F.Cu at (115.9, 82.6)
- added R12: MBA02040C7320FRP00, Resistor_THT:R_Axial_DIN0204_L3.6mm_D1.6mm_P5.08mm_Horizontal, F.Cu at (110.8, 85.2)
- added R13: WLBR050FET, Resistor_THT:R_Axial_DIN0411_L9.9mm_D3.6mm_P12.70mm_Horizontal, F.Cu at (116.2, 114.3)
- added R15: CRCW0402100KFKED, extracted:RESC1005X40N, F.Cu at (113.2, 116.6)
- added R16: RN55D3202FB14, Resistor_THT:R_Axial_DIN0207_L6.3mm_D2.5mm_P7.62mm_Horizontal, F.Cu at (120.2, 123.1)
- added R17: CF14JT620R, Resistor_THT:R_Axial_DIN0207_L6.3mm_D2.5mm_P7.62mm_Horizontal, F.Cu at (133.6, 121.5)
- added R9: WLBR050FET, Resistor_THT:R_Axial_DIN0411_L9.9mm_D3.6mm_P12.70mm_Horizontal, F.Cu at (139.1, 116.2)
- moved Q1 31.2 mm to (109.2, 104.0)
- moved R3 30.2 mm to (112.7, 104.7)
- moved C9 19.5 mm to (121.3, 96.2), turned to 0 degrees
- moved C17 19.4 mm to (124.7, 96.3), turned to 180 degrees
- moved R14 19.0 mm to (131.2, 99.8), turned to 90 degrees
- moved R7 18.9 mm to (116.2, 100.3), turned to 0 degrees
- moved R8 17.9 mm to (118.7, 103.3), turned to 0 degrees
- moved C10 17.9 mm to (128.1, 97.0), turned to 180 degrees
- moved R4 17.8 mm to (114.2, 103.5), turned to -90 degrees
- moved C7 17.3 mm to (116.7, 98.3)
- moved C13 16.5 mm to (128.7, 110.0)
- moved C1 16.4 mm to (118.2, 110.1)
- moved C12 15.1 mm to (127.0, 99.2), turned to 180 degrees
- moved R1 13.2 mm to (116.8, 102.2), turned to -90 degrees
- moved C19 12.9 mm to (129.4, 103.3), turned to 180 degrees
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- renumbered C19 to C10, C20 to C11, C13 to C12, C2 to C13, C18 to C14, C14 to C15, C6 to C16, C21 to C17, C4 to C18, C10 to C19, C3 to C2, C7 to C20, C11 to C21, C5 to C3, C8 to C4, C9 to C5, C12 to C6, C15 to C7, C16 to C8, C17 to C9, R5 to R1, R3 to R14, R4 to R18, R11 to R19, R8 to R2, R12 to R20, R1 to R3, R2 to R4, R6 to R5, R7 to R6, R10 to R7, R9 to R8
Connections:
- net COMP renamed Net-(C12-Pad2)
- net COMP-2 renamed Net-(C15-Pad2)
- A1 pad GND2: BATT- -> GND
- A1 pad VIN: ISP-2 -> V5+
- C1 pad 1: BATT- -> BATT+
- C1 pad 2: BATT+ -> GND
- C10 pad 1: BATT- -> GND
- C11 pad 1: BATT- -> GND
- C13 pad 1: BATT- -> V15+
- C13 pad 2: ISP -> GND
- C16 pad 1: BATT- -> GND
- C16 pad 2: ISP -> V15+
- C18 pad 1: BATT- -> V5+
- C18 pad 2: ISP-2 -> GND
- C19 pad 1: BATT- -> GND
- C19 pad 2: ISP -> V15+
- C2 pad 1: BATT- -> BATT+
- C2 pad 2: BATT+ -> GND
- C20 pad 1: BATT- -> GND
- C20 pad 2: ISP-2 -> V5+
- C21 pad 1: BATT- -> GND
- C21 pad 2: ISP-2 -> V5+
- C22 pad 1: BATT- -> GND
- C22 pad 2: ISP-2 -> V5+
- C23 pad 1: BATT- -> GND
- C3 pad 1: BATT- -> GND
- C4 pad 1: BATT- -> GND
- C5 pad 1: BATT- -> GND
- C6 pad 1: BATT- -> GND
- C7 pad 1: BATT- -> GND
- J10 pad 1: BATT- -> GND
- J5 pad 1: BATT- -> GND
- J5 pad 2: BATT- -> GND
- J5 pad 3: BATT- -> GND
- J5 pad 4: BATT- -> GND
- J5 pad 5: BATT- -> GND
- J5 pad 6: BATT- -> GND
- J6 pad 1: ISP-2 -> V5+
- J6 pad 2: ISP-2 -> V5+
- J6 pad 3: ISP-2 -> V5+
- J6 pad 4: ISP-2 -> V5+
- J6 pad 5: ISP-2 -> V5+
- J6 pad 6: ISP-2 -> V5+
- J7 pad 1: ISP-2 -> V5+
- J7 pad 2: BATT- -> GND
- J8 pad 1: BATT- -> GND
- J8 pad 2: ISP -> V15+
- R1 pad 1: BATT- -> GND
- R14 pad 1: BATT- -> GND
- R18 pad 1: BATT- -> GND
- R19 pad 2: ISP-2 -> V5+
- R2 pad 1: BATT- -> GND
- R20 pad 2: ISP-2 -> V5+
- R4 pad 1: BATT- -> GND
- R6 pad 1: BATT- -> GND
- R7 pad 1: BATT- -> GND
- U1 pad 11: ISP -> Net-(R9-Pad2)
- U1 pad 12: ISP -> Net-(R9-Pad2)
- U1 pad 13: ISP -> V15+
- U1 pad 14: unconnected-(U1-Pad14) -> Net-(R10-Pad1)
- U1 pad 17: BATT- -> GND
- U1 pad 2: BATT- -> GND
- U1 pad 22: BATT- -> GND
- U1 pad 23: BATT- -> GND
- U1 pad 3: BATT- -> GND
- U1 pad 4: BATT- -> GND
- U1 pad 5: BATT- -> GND
- U1 pad 9: BATT- -> GND
- U2 pad 11: ISP-2 -> Net-(R13-Pad2)
- U2 pad 12: ISP-2 -> Net-(R13-Pad2)
- U2 pad 13: ISP-2 -> V5+
- U2 pad 14: unconnected-(U2-Pad14) -> Net-(R15-Pad1)
- U2 pad 17: BATT- -> GND
- U2 pad 2: BATT- -> GND
- U2 pad 22: BATT- -> GND
- U2 pad 23: BATT- -> GND
- U2 pad 3: BATT- -> GND
- U2 pad 4: BATT- -> GND
- U2 pad 5: BATT- -> GND
- U2 pad 9: BATT- -> GND
- U3 pad 10: BATT- -> GND
- U3 pad 11: BATT- -> GND
- U3 pad 12: BATT- -> GND
- U3 pad 13: BATT- -> GND
- U3 pad 2: ISP-2 -> V5+
- U3 pad 5: BATT- -> GND
- U3 pad 6: BATT- -> GND
- U3 pad 7: BATT- -> GND
- U3 pad 8: BATT- -> GND
- U3 pad 9: BATT- -> GND
- U4 pad 3: BATT- -> GND
Routing:
- net GND: track 0.00 -> 142.2 mm, vias 0 -> 34
- net BATT-: track 123.0 -> 0.00 mm, vias 30 -> 0
- net ISP-2: track 75.6 -> 0.00 mm, vias 7 -> 0
- net V5+: track 0.00 -> 70.5 mm, vias 0 -> 8
- net V15+: track 0.00 -> 60.6 mm, vias 0 -> 1
- net BATT+: track 122.1 -> 62.2 mm, vias 3 -> 0
- net ISP: track 33.6 -> 0.00 mm
- net A4: track 17.9 -> 50.9 mm, vias 0 -> 1
- net Net-(R10-Pad1): track 0.00 -> 30.7 mm, vias 0 -> 2
- net Net-(R9-Pad2): track 0.00 -> 19.4 mm
- net Net-(R13-Pad2): track 0.00 -> 15.7 mm
- net Net-(R15-Pad1): track 0.00 -> 13.8 mm
- net Net-(Q1-Pad1): track 16.3 -> 5.15 mm
- net Net-(R16-Pad1): track 0.00 -> 6.40 mm
- net SW1: track 14.9 -> 10.2 mm
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- added copper zone on B.Cu, net GND
- added copper zone on F.Cu, net GND
- added copper zone on In2.Cu, net V5+
- removed copper zone on B.Cu, net BATT-
- removed copper zone on F.Cu, net BATT-
- removed copper zone on In2.Cu, net ISP-2
Other:
- board text added: "ALANIZER SHIELD v2.0 Daphne Chevalier License: CC BY 4.0"
- board text removed: "ALANIZER SHIELD v1.0 Daphne Chevalier License: CC BY 4.0"
